Commit message: update

File: leelawadee_description/urdf/leelawadee_base/leelawadee_base.xacro (robot description, xacro)
@@ -1,3 +1,144 @@
 <?xml version="1.0"?>
-<robot name="leelawadee_robot" xmlns:xacro="http://ros.org/wiki/xacro">
+<robot name="leelawadee_robot"
+    xmlns:xacro="http://ros.org/wiki/xacro">
+    <xacro:include filename="$(find leelawadee_description)/urdf/materials.xacro"/>
+    <link name="base_link">
+        <visual>
+            <origin xyz="0 0 -0.055" rpy="1.5707 0 -1.5707" />
+            <geometry>
+                <mesh filename="package://leelawadee_description/urdf/leelawadee_base/meshes/chessis.STL" scale="1 1 1" />
+            </geometry>
+            <material name="green"/>
+        </visual>
+        <collision>
+            <origin xyz="0 0 -0.055" rpy="1.5707 0 -1.5707" />
+            <geometry>
+                <mesh filename="package://leelawadee_description/urdf/leelawadee_base/meshes/chessis.STL" scale="1 1 1" />
+            </geometry>
+            <surface>
+                <friction>
+                    <ode>
+                        <mu>0</mu>
+                        <mu2>0</mu2>
+                        <slip1>1.0</slip1>
+                        <slip2>1.0</slip2>
+                    </ode>
+                </friction>
+            </surface>
+            <material name="green"/>
+        </collision>
+        <inertial>
+            <mass value="15.0"/>
+            <origin xyz="0.0 -0.15 0.1" rpy=" 0 0 0"/>
+            <inertia ixx="0.1" ixy="0" ixz="0" iyy="0.1" iyz="0" izz="0.1" />
+        </inertial>
+    </link>
+    <joint name="left_wheel_joint" type="continuous">
+        <origin xyz="0 0.2 0" rpy="0 0 0"/>
+        <child link="left_wheel"/>
+        <parent link="base_link"/>
+        <axis xyz="0 0 1" rpy="0 0 0"/>
+        <limit effort="10000" velocity="1000"/>
+        <joint_properties damping="1.0" friction="1.0"/>
+    </joint>
+    <joint name="right_wheel_joint" type="continuous">
+        <origin xyz="0 -0.2 0" rpy="0 0 3.14159"/>
+        <child link="right_wheel"/>
+        <parent link="base_link"/>
+        <axis xyz="0 0 1" rpy="0 0 0"/>
+        <limit effort="10000" velocity="1000"/>
+        <joint_properties damping="1.0" friction="1.0"/>
+    </joint>
+    <link name="left_wheel">
+        <visual>
+            <origin xyz="0 0 0" rpy="0 0 0" />
+            <geometry>
+                <mesh filename="package://leelawadee_description/urdf/leelawadee_base/meshes/LWheel.STL" scale="1 1 1" />
+            </geometry>
+            <material name="orange"/>
+        </visual>
+        <collision>
+            <origin xyz="0 0 0" rpy="0 0 0" />
+            <geometry>
+                <mesh filename="package://leelawadee_description/urdf/leelawadee_base/meshes/LWheel.STL" scale="1 1 1" />
+            </geometry>
+            <material name="orange"/>
+        </collision>
+        <inertial>
+            <mass value="5"/>
+            <inertia ixx=".1" ixy="0.0" ixz="0.0" iyy=".1" iyz="0.0" izz=".1"/>
+        </inertial>
+    </link>
+    <link name="right_wheel">
+        <visual>
+            <origin xyz="0 0 0" rpy="0 0 0" />
+            <geometry>
+                <mesh filename="package://leelawadee_description/urdf/leelawadee_base/meshes/RWheel.STL" scale="1 1 1" />
+            </geometry>
+            <material name="orange"/>
+        </visual>
+        <collision>
+            <origin xyz="0 0 0" rpy="0 0 0" />
+            <geometry>
+                <mesh filename="package://leelawadee_description/urdf/leelawadee_base/meshes/RWheel.STL" scale="1 1 1" />
+            </geometry>
+            <material name="orange"/>
+        </collision>
+        <inertial>
+            <mass value="5"/>
+            <inertia ixx=".1" ixy="0.0" ixz="0.0" iyy=".1" iyz="0.0" izz=".1"/>
+        </inertial>
+    </link>
+    <joint name="laser_fixed" type="fixed">
+        <origin xyz="0.15 0 .1" rpy="0 0 0"/>
+        <parent link="base_link"/>
+        <child link="laser_link"/>
+    </joint>
+    <link name="laser_link">
+        <visual>
+            <origin xyz="-0.03 0.01 -0.005" rpy="-1.5707 0 -1.5707" />
+            <geometry>
+                <mesh filename="package://leelawadee_description/urdf/leelawadee_base/meshes/LidarG4.stl" scale="0.001 0.001 0.001" />
+            </geometry>
+            <material name="blue"/>
+        </visual>
+        <collision>
+            <origin xyz="-0.03 0.01 -0.005" rpy="-1.5707 0 -1.5707" />
+            <geometry>
+                <mesh filename="package://leelawadee_description/urdf/leelawadee_base/meshes/LidarG4.stl" scale="0.001 0.001 0.001" />
+            </geometry>
+            <material name="blue"/>
+        </collision>
+        <inertial>
+            <mass value="0.3" />
+            <origin xyz="0 0 0" rpy="0 0 0"/>
+            <inertia ixx="0.01" ixy="0" ixz="0" iyy="0.01" iyz="0" izz="0.01" />
+        </inertial>
+    </link>
+    <joint name="imu_fixed" type="fixed">
+        <origin xyz="-0.1 0 0.05" rpy="0 0 0"/>
+        <parent link="base_link"/>
+        <child link="imu_link"/>
+    </joint>
+    <link name="imu_link">
+        <visual>
+            <origin xyz="0 0 0" rpy="0 0 0" />
+            <geometry>
+                <box size="0.02 0.02 0.02"/>
+            </geometry>
+            <material name="blue"/>
+        </visual>
+        <collision>
+            <origin xyz="0 0 0" rpy="0 0 0" />
+            <geometry>
+                <box size="0.02 0.02 0.02"/>
+            </geometry>
+            <material name="blue"/>
+        </collision>
+        <inertial>
+            <mass value="1e-5" />
+            <origin xyz="0 0 0" rpy="0 0 0"/>
+            <inertia ixx="1e-6" ixy="0" ixz="0" iyy="1e-6" iyz="0" izz="1e-6" />
+        </inertial>
+    </link>
 </robot>
